File: lark.sch (KiCad schematic (older format))
At the start: 33 parts, among them J1 CONN1, J11 CONN1, J3 Conn_01x05-Connector_Generic, J6 Conn_01x05-Connector_Generic, U6 BMI088

Commit message: change I2C pullups to 1k2
Parts:
- R18, R19: value 10k -> 1k2
Changed lines of the file:
@@
 P 4450 5900
 F 0 "R18" H 4520 5946 50  0000 L CNN
-F 1 "10k" H 4520 5855 50  0000 L CNN
+F 1 "1k2" H 4520 5855 50  0000 L CNN
 F 2 "Resistor_SMD:R_0805_2012Metric_Pad1.15x1.40mm_HandSolder" V 4380 5900 50  0001 C CNN
 F 3 "~" H 4450 5900 50  0001 C CNN
@@
 P 4800 5900
 F 0 "R19" H 4870 5946 50  0000 L CNN
-F 1 "10k" H 4870 5855 50  0000 L CNN
+F 1 "1k2" H 4870 5855 50  0000 L CNN
 F 2 "Resistor_SMD:R_0805_2012Metric_Pad1.15x1.40mm_HandSolder" V 4730 5900 50  0001 C CNN
 F 3 "~" H 4800 5900 50  0001 C CNN
